Commit message: update slam

File: description/urdf/robot.urdf (robot description, URDF)
Before this commit: robot robot, 7 links, 6 joints
Links:
- removed link base_link
- added link base_footprint; collision cylinder length=0.001 radius=0.25; visual cylinder length=0.001 radius=0.25
- added link laser; collision cylinder length=0.025 radius=0.03; visual cylinder length=0.025 radius=0.03
Joints:
- added joint laser_to_lidar: type fixed, parent lidar, child laser, origin xyz=0 0 0 rpy=0 0 3.14159265
- joint base_to_base_link_joint: parent base_link -> base_footprint

Commit message: update

File: description/urdf/robot.urdf (robot description, URDF)
Before this commit: robot robot, 8 links, 7 joints
Joints:
- joint lidar_to_base_joint: origin xyz=0.15 0 0.1125 rpy=0 0 3.14159265 -> xyz=0.15 0 0.1125 rpy=0 0 0
